Commit message: add laserscanner to robot model

File: urdf/mobrob_move.urdf (robot description, URDF)
Before this commit: robot mobrob, 10 links, 9 joints
Links:
- added link laser
Joints:
- added joint base_to_laser: type fixed, parent base_link, child laser, origin xyz=0.055 0 0.06 rpy=0 0 3.14159

Commit message: add laserscanner to model with visuals

File: urdf/mobrob_move.urdf (robot description, URDF)
Before this commit: robot mobrob, 11 links, 10 joints
Links:
- link laser: geometry visual cylinder length=0.03 radius=0.04
