Commit message: add screenshot of rviz

File: urdf/mobrob_fixed.urdf (robot description, URDF)
Before this commit: robot mobrob_fixed, 10 links, 9 joints
Links:
- added link laser; visual cylinder length=0.03 radius=0.04
Joints:
- added joint base_to_laser: type fixed, parent base_link, child laser, origin xyz=0.055 0 0.06 rpy=0 0 3.14159
