Commit message: fix laser orientation

File: urdf/mobrob_move.xacro (robot description, xacro)
@@ -83,5 +83,5 @@
     <parent link="base_link"/>
     <child link="laser"/>
-    <origin rpy="0 0 0" xyz="0.055 0 0.06"/>
+    <origin rpy="0 0 3.14159" xyz="0.055 0 0.06"/>
   </joint>
   <link name="right_front_wheel">

Commit message: landmark extraction and visualisation finished

File: urdf/mobrob_move.xacro (robot description, xacro)
@@ -84,5 +84,5 @@
     <parent link="base_link"/>
     <child link="laser"/>
-    <origin rpy="0 0 3.14159" xyz="0.055 0 0.06"/>
+    <origin rpy="0 0 1.57075" xyz="0.055 0 0.06"/>
   </joint>
   <link name="right_front_wheel">

Commit message: fix orientation of laser

File: urdf/mobrob_move.xacro (robot description, xacro)
@@ -84,5 +84,6 @@
     <parent link="base_link"/>
     <child link="laser"/>
-    <origin rpy="0 0 1.57075" xyz="0.055 0 0.06"/>
+    <!--<origin rpy="0 0 1.57075" xyz="0.055 0 0.06"/>-->
+    <origin rpy="0 0 0" xyz="0.055 0 0.06"/>
   </joint>
   <link name="right_front_wheel">

Commit message: fix lidar orientation and material issue

File: urdf/mobrob_move.xacro (robot description, xacro)
@@ -1,6 +1,7 @@
 <?xml version="1.0"?>
 <robot name="mobrob" xmlns:xacro="http://www.ros.org/wiki/xacro">
-  <!--<xacro:include filename="$(find myrobot_model)/urdf/mobrob_gpu.gazebo" />-->
-  <xacro:include filename="$(find myrobot_model)/urdf/mobrob.gazebo" />
+  <xacro:include filename="$(find myrobot_model)/urdf/mobrob_gpu.gazebo" />
+  <!--<xacro:include filename="$(find myrobot_model)/urdf/mobrob.gazebo" />-->
+  <xacro:include filename="$(find myrobot_model)/urdf/materials.urdf.xacro" />
   <link name="base_footprint"></link>
   <joint name="base_link_joint" type="fixed">
@@ -85,5 +86,5 @@
     <child link="laser"/>
     <!--<origin rpy="0 0 1.57075" xyz="0.055 0 0.06"/>-->
-    <origin rpy="0 0 0" xyz="0.055 0 0.06"/>
+    <origin rpy="0 0 ${-pi}" xyz="0.055 0 0.06"/>
   </joint>
   <link name="right_front_wheel">

Commit message: add camera to urdf model and integrate feedback from attiny to joint state publisher

File: urdf/mobrob_move.xacro (robot description, xacro)
@@ -314,3 +314,83 @@
     <limit effort="1000.0" lower="0" upper="0.11" velocity="0.5"/>
   </joint>
+  <link name="camera_servo">
+    <visual>
+      <origin rpy="0 0 0" xyz="-0.01 0.015 0.008"/>
+      <geometry>
+        <box size="0.035 0.03 0.016"/>
+      </geometry>
+    </visual>
+    <collision>
+      <origin rpy="0 0 0" xyz="-0.01 0.015 0.008"/>
+      <geometry>
+        <box size="0.03 0.035 0.016"/>
+      </geometry>
+    </collision>
+    <inertial>
+      <mass value="0.012"/>
+      <inertia
+        ixx="0.000000732" ixy="0.0" ixz="0.0"
+        iyy="0.000002118" iyz="0.0"
+        izz="0.00000166"/>
+    </inertial>
+  </link>
+  <joint name="base_to_camera_servo_joint" type="fixed">
+    <parent link="base_link"/>
+    <child link="camera_servo"/>
+    <origin rpy="0 0 0" xyz="0.21 0 0.27"/>
+  </joint>
+  <link name="camera_base">
+    <visual>
+      <origin rpy="0 0 0" xyz="0.02 0 -0.02"/>
+      <geometry>
+        <box size="0.004 0.04 0.04"/>
+      </geometry>
+    </visual>
+    <collision>
+      origin rpy="0 0 0" xyz="-0.01 0.015 0.01"/>
+      <geometry>
+        <box size="0.002 0.04 0.04"/>
+      </geometry>
+    </collision>
+    <inertial>
+      <mass value="0.012"/>
+      <inertia
+        ixx="0.000000732" ixy="0.0" ixz="0.0"
+        iyy="0.000002118" iyz="0.0"
+        izz="0.00000166"/>
+    </inertial>
+  </link>
+  <joint name="camera_servo_to_camera_base_joint" type="revolute">
+    <parent link="camera_servo"/>
+    <child link="camera_base"/>
+    <origin rpy="0 1.57075 3.14159" xyz="0 0 0"/>
+    <axis xyz="0 1 0"/>
+    <limit effort="1000.0" lower="0.69" upper="3.14159" velocity="0.5"/>
+  </joint>
+  <link name="camera_center">
+    <visual>
+      <origin rpy="0 1.57075 0" xyz="0.01 0 0"/>
+      <geometry>
+        <cylinder length="0.02" radius="0.006"/>
+      </geometry>
+    </visual>
+    <collision>
+      <origin rpy="0 0 0" xyz="-0.01 0 0"/>
+      <geometry>
+        <cylinder length="0.02" radius="0.006"/>
+      </geometry>
+    </collision>
+    <inertial>
+      <mass value="0.012"/>
+      <inertia
+        ixx="0.000000732" ixy="0.0" ixz="0.0"
+        iyy="0.000002118" iyz="0.0"
+        izz="0.00000166"/>
+    </inertial>
+  </link>
+  <joint name="camera_base_to_camera_center_joint" type="fixed">
+    <parent link="camera_base"/>
+    <child link="camera_center"/>
+    <origin rpy="0 0 0" xyz="0.02 0 -0.02"/>
+  </joint>
 </robot>

Commit message: add basic camera to gazebo

File: urdf/mobrob_move.xacro (robot description, xacro)
@@ -392,5 +392,5 @@
     <parent link="camera_base"/>
     <child link="camera_center"/>
-    <origin rpy="0 0 0" xyz="0.02 0 -0.02"/>
+    <origin rpy="3.14159 0 0" xyz="0.02 0 -0.02"/>
   </joint>
 </robot>

Commit message: attiny gazebo plugin wip

File: urdf/mobrob_move.xacro (robot description, xacro)
@@ -255,6 +255,7 @@
     <child link="gripper_base"/>
     <axis xyz="0 0 1"/>
-    <limit effort="1000.0" lower="-0.11" upper="0" velocity="0.5"/>
+    <limit effort="1000.0" lower="-0.15" upper="0" velocity="0.5"/>
     <origin rpy="0 0 0" xyz="0.075 0 0"/>
+    <dynamics damping="0.01" friction="0.1"/>
   </joint>
   <link name="right_finger">
@@ -262,5 +263,5 @@
       <origin rpy="0 0 0" xyz="0 -0.006  0"/>
       <geometry>
-        <box size="0.04 0.012 0.025"/>
+        <box size="0.08 0.012 0.025"/>
       </geometry>
     </visual>
@@ -268,5 +269,5 @@
       <origin rpy="0 0 0" xyz="0 -0.006  0"/>
       <geometry>
-        <box size="0.04 0.012 0.025"/>
+        <box size="0.08 0.012 0.025"/>
       </geometry>
     </collision>
@@ -285,4 +286,5 @@
     <axis xyz="0 1 0"/>
     <limit effort="1000.0" lower="-0.11" upper="0" velocity="0.5"/>
+    <dynamics damping="0.01" friction="0.1"/>
   </joint>
   <link name="left_finger">
@@ -290,5 +292,5 @@
       <origin rpy="0 0 0" xyz="0 0.006 0"/>
       <geometry>
-        <box size="0.04 0.012 0.025"/>
+        <box size="0.08 0.012 0.025"/>
       </geometry>
     </visual>
@@ -296,5 +298,5 @@
       <origin rpy="0 0 0" xyz="0 0.006 0"/>
       <geometry>
-        <box size="0.04 0.012 0.025"/>
+        <box size="0.08 0.012 0.025"/>
       </geometry>
     </collision>
@@ -313,4 +315,5 @@
     <axis xyz="0 1 0"/>
     <limit effort="1000.0" lower="0" upper="0.11" velocity="0.5"/>
+    <dynamics damping="0.01" friction="0.1"/>
   </joint>
   <link name="camera_servo">

Commit message: finish gazebo plugin for gripper

File: urdf/mobrob_move.xacro (robot description, xacro)
@@ -218,9 +218,9 @@
     </collision>
     <inertial>
-      <mass value="0.28"/>
-      <inertia
-        ixx="0.001154" ixy="0.0" ixz="0.0"
-        iyy="0.0007792" iyz="0.0"
-        izz="0.0004165"/>
+      <mass value="0.028"/>
+      <inertia
+        ixx="0.0001154" ixy="0.0" ixz="0.0"
+        iyy="0.00007792" iyz="0.0"
+        izz="0.00004165"/>
     </inertial>
   </link>
@@ -244,9 +244,9 @@
     </collision>
     <inertial>
-      <mass value="0.228"/>
-      <inertia
-        ixx="0.001249" ixy="0.0" ixz="0.0"
-        iyy="0.00009213" iyz="0.0"
-        izz="0.001218"/>
+      <mass value="0.0228"/>
+      <inertia
+        ixx="0.0001249" ixy="0.0" ixz="0.0"
+        iyy="0.000009213" iyz="0.0"
+        izz="0.0001218"/>
     </inertial>
   </link>
@@ -255,7 +255,6 @@
     <child link="gripper_base"/>
     <axis xyz="0 0 1"/>
-    <limit effort="1000.0" lower="-0.15" upper="0" velocity="0.5"/>
+    <limit effort="1000.0" lower="-0.12" upper="0" velocity="0.5"/>
     <origin rpy="0 0 0" xyz="0.075 0 0"/>
-    <dynamics damping="0.01" friction="0.1"/>
   </joint>
   <link name="right_finger">
@@ -286,5 +285,4 @@
     <axis xyz="0 1 0"/>
     <limit effort="1000.0" lower="-0.11" upper="0" velocity="0.5"/>
-    <dynamics damping="0.01" friction="0.1"/>
   </joint>
   <link name="left_finger">
@@ -315,5 +313,4 @@
     <axis xyz="0 1 0"/>
     <limit effort="1000.0" lower="0" upper="0.11" velocity="0.5"/>
-    <dynamics damping="0.01" friction="0.1"/>
   </joint>
   <link name="camera_servo">
